File: Schematic/CoolCook/LowTemp_board_2.sch (EAGLE design)
At the start: 11 parts, among them SW2 EC11B-V

Commit message: Update schematic in two boards (test and work great) Reverse rotation in arduino program
Parts:
- C1, C2: device rcl:C-EU050-024X044 -> rcl:C-EU050-025X075
Changed lines of the file:
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@@
 <part name="AGND3" library="supply1" deviceset="AGND" device=""/>
 <part name="AGND4" library="supply1" deviceset="AGND" device=""/>
-<part name="C1" library="rcl" deviceset="C-EU" device="050-024X044" value="0,1µF"/>
-<part name="C2" library="rcl" deviceset="C-EU" device="050-024X044" value="0,1µF"/>
+<part name="C1" library="rcl" deviceset="C-EU" device="050-025X075" value="0,1µF"/>
+<part name="C2" library="rcl" deviceset="C-EU" device="050-025X075" value="0,1µF"/>
 <part name="R1" library="resistor" deviceset="R-EU_" device="0207/7" value="10kΩ"/>
 <part name="R2" library="resistor" deviceset="R-EU_" device="0207/7" value="10kΩ"/>
